Commit message: map+slam
map+finder v1

File: mobile_robot/urdf/lidar.xacro (robot description, xacro)
@@ -44,5 +44,5 @@
             <range>
             <min>0.20</min>
-            <max>6</max>
+            <max>12</max>
             <resolution>0.015</resolution>
             </range>

File: mobile_robot/urdf/rover.urdf copy.xacro (robot description, xacro)
@@ -1,11 +1,5 @@
 <?xml version="1.0"?>
 <robot xmlns:xacro="http://www.ros.org/wiki/xacro" name="rover">
-<link name="map"/>
-<link name="odom"/>
-<joint name="my_joint" type="fixed">
-    <origin xyz="0 0 0" rpy="0 0 0"/>
-    <parent link="odom"/>
-    <child link="map"/>
- </joint>
+<link name="base_footprint"/>
 <xacro:property name="constant" value="1/12"/>
 <xacro:property name="mass" value="1.0"/>
@@ -40,5 +34,5 @@
 <joint name="base_joint" type="fixed">
     <origin xyz="0.0 0.0 0.135" rpy="0.0 0.0 0.0"/>
-    <parent link="odom"/>
+    <parent link="base_footprint"/>
     <child link="base_link"/>
     <axis xyz="0.0 0.0 0.0"/>
@@ -89,5 +83,5 @@
 <gazebo>
   <plugin name="skid_steer_drive_controller" filename="libgazebo_ros_skid_steer_drive.so">
-    <updateRate>5.0</updateRate>
+    <updateRate>10.0</updateRate>
     <robotNamespace>/</robotNamespace>
     <leftFrontJoint>wheel_front_left_joint</leftFrontJoint>
@@ -101,7 +95,4 @@
     <topicName>cmd_vel</topicName>
     <broadcastTF>true</broadcastTF>
-    <odometryTopic>odom</odometryTopic>
-    <odometryFrame>odom</odometryFrame>
-    <robotBaseFrame>base_footprint</robotBaseFrame>
   </plugin>
 </gazebo>
